Commit message: #add new features: pick and place

File: omtb_description/omtb_description/urdf/open_manipulator_with_tb3.gazebo.xacro (robot description, xacro)
@@ -29,4 +29,8 @@
   <!-- gripper_link_sub -->
   <RefLink ref="gripper_link_sub"/>
+  <!-- end effector link -->
+  <gazebo reference="end_effector_link">
+    <material>Gazebo/Red</material>
+  </gazebo>
   <!-- ros_control plugin -->
   <gazebo>

File: omtb_description/omtb_description/urdf/open_manipulator_with_tb3_waffle.urdf.xacro (robot description, xacro)
@@ -1,5 +1,5 @@
 <?xml version="1.0"?>
 <!-- Open_Manipulator Chain -->
-<robot name="om_with_tb3" xmlns:xacro="http://ros.org/wiki/xacro">
+<robot name="robot" xmlns:xacro="http://ros.org/wiki/xacro">
   <xacro:arg name="use_robot_name"    default="robot1"/>
   <xacro:property name="use_robot_name" value="$(arg use_robot_name)" />
@@ -249,4 +249,25 @@
   <!-- Transmission 6 -->
   <xacro:SimpleTransmission n="6" joint="gripper_sub" />
+  <!-- end effector joint -->
+  <joint name="end_effector_joint" type="fixed">
+    <origin xyz="0.126 0.0 0.0" rpy="0 0 0"/>
+    <parent link="link5"/>
+    <child link="end_effector_link"/>
+  </joint>
+  <!-- end effector link -->
+  <link name="end_effector_link">
+<!--    <visual>
+      <origin xyz="0 0 0" rpy="0 0 0"/>
+      <geometry>
+        <box size="0.001 0.010 0.001" />
+      </geometry>
+      <material name="red"/>
+     </visual>-->
+    <inertial>
+      <origin xyz="0.0 0.0 0.0" rpy="0 0 0"/>
+      <mass value="0.001"/>
+      <inertia ixx="0.001" ixy="0.0" ixz="0.0" iyy="0.001" iyz="0.0" izz="0.001" />
+    </inertial>
+  </link>
   <joint name="eye_in_hand_joint" type="fixed">
     <origin xyz="0.03 0 0.07" rpy="0 0 0"/>

File: omtb_description/turtlebot3_description/urdf/turtlebot3_waffle.gazebo.xacro (robot description, xacro)
@@ -10,6 +10,6 @@
   </gazebo>
   <gazebo reference="wheel_left_link">
-    <mu1>1</mu1>
-    <mu2>1</mu2>
+    <mu1>0.5</mu1>
+    <mu2>0.5</mu2>
     <kp>1000000.0</kp>
     <kd>100.0</kd>
@@ -20,6 +20,6 @@
   </gazebo>
   <gazebo reference="wheel_right_link">
-    <mu1>1</mu1>
-    <mu2>1</mu2>
+    <mu1>0.5</mu1>
+    <mu2>0.5</mu2>
     <kp>1000000.0</kp>
     <kd>100.0</kd>
@@ -30,6 +30,6 @@
   </gazebo>
   <gazebo reference="caster_back_right_link">
-    <mu1>1</mu1>
-    <mu2>1</mu2>
+    <mu1>0.5</mu1>
+    <mu2>0.5</mu2>
     <kp>1000000.0</kp>
     <kd>100.0</kd>
@@ -39,6 +39,6 @@
   </gazebo>
   <gazebo reference="caster_back_left_link">
-    <mu1>1</mu1>
-    <mu2>1</mu2>
+    <mu1>0.5</mu1>
+    <mu2>0.5</mu2>
     <kp>1000000.0</kp>
     <kd>100.0</kd>

File: omtb_description/turtlebot3_description/urdf/turtlebot3_waffle_for_open_manipulator.urdf.xacro (robot description, xacro)
@@ -186,10 +186,10 @@
   </joint>
   <link name="camera_link">
-    <visual>
+<!--    <visual>
      <origin xyz="0 0 0" rpy="1.57 0 1.57"/>
       <geometry>
        <mesh filename="package://omtb_description/turtlebot3_description/meshes/sensors/r200.dae" />
       </geometry>
-    </visual>
+    </visual>-->
   </link>
   <joint name="camera_rgb_joint" type="fixed">
