Commit message: # add multi-line lidar

File: omtb_description/turtlebot3_description/urdf/turtlebot3_waffle.gazebo.xacro (robot description, xacro)
@@ -1,5 +1,5 @@
 <?xml version="1.0"?>
 <robot name="turtlebot3_waffle_sim" xmlns:xacro="http://ros.org/wiki/xacro">
-  <xacro:arg name="laser_visual"  default="true"/>
+  <xacro:arg name="laser_visual"  default="false"/>
   <xacro:arg name="camera_visual" default="false"/>
   <xacro:arg name="imu_visual"    default="false"/>
@@ -117,5 +117,5 @@
             <resolution>1</resolution>
             <min_angle>0.0</min_angle>
-            <max_angle>6.28319</max_angle>
+            <max_angle>6.283185</max_angle>
           </horizontal>
         </scan>
@@ -134,4 +134,46 @@
         <topicName>scan</topicName>
         <frameName>base_scan</frameName>
+      </plugin>
+    </sensor>
+  </gazebo>
+  <gazebo reference="multi_base_scan">
+    <sensor type="ray" name="VLP16">
+      <pose>0 0 0 0 0 0</pose>
+      <visualize>false</visualize>
+      <update_rate>20</update_rate>
+      <ray>
+        <scan>
+          <horizontal>
+            <samples>360</samples>
+            <resolution>1</resolution>
+            <min_angle>0.0</min_angle>
+            <max_angle>6.283185</max_angle>
+          </horizontal>
+          <vertical>
+            <samples>16</samples>
+<!--            <samples>9</samples>-->
+            <resolution>1</resolution>
+<!--            <min_angle>-0.017453</min_angle>-->
+            <min_angle>-0.523599</min_angle>
+            <max_angle>0.523599</max_angle>
+          </vertical>
+        </scan>
+        <range>
+          <min>0.3</min>
+          <max>3.5</max>
+          <resolution>0.02</resolution>
+        </range>
+        <noise>
+          <type>gaussian</type>
+          <mean>0.0</mean>
+          <stddev>0.01</stddev>
+        </noise>
+      </ray>
+      <plugin name="gazebo_ros_laser_controller" filename="libgazebo_ros_velodyne_laser.so">
+        <topicName>points2</topicName>
+        <frameName>multi_base_scan</frameName>
+        <min_range>0.3</min_range>
+        <max_range>3.5</max_range>
+        <gaussianNoise>0.01</gaussianNoise>
       </plugin>
     </sensor>

File: omtb_description/turtlebot3_description/urdf/turtlebot3_waffle_for_open_manipulator.urdf.xacro (robot description, xacro)
@@ -173,5 +173,5 @@
     </collision>
     <inertial>
-      <mass value="1.14" />
+      <mass value="0.1" />
       <origin xyz="0 0 0" />
       <inertia ixx="0.001" ixy="0.0" ixz="0.0"
@@ -179,4 +179,52 @@
                izz="0.001" />
     </inertial>
+  </link>
+  <joint name="multi_base_mount_joint" type="fixed">
+    <parent link="base_link"/>
+    <child link="multi_base_scan"/>
+    <origin xyz="-0.024 0 0.122" rpy="0 0 0"/>
+  </joint>
+  <link name="multi_base_scan">
+    <inertial>
+      <mass value="0.1"/>
+      <origin xyz="0 0 0.03585"/>
+      <inertia ixx="1" ixy="0" ixz="0"
+        iyy="1" iyz="0"
+        izz="1"/>
+    </inertial>
+    <visual>
+      <geometry>
+        <mesh filename="package://velodyne_description/meshes/VLP16_base_1.dae" scale="0.5 0.5 0.5"/>
+      </geometry>
+    </visual>
+    <visual>
+      <geometry>
+        <mesh filename="package://velodyne_description/meshes/VLP16_base_2.dae" scale="0.5 0.5 0.5"/>
+      </geometry>
+    </visual>
+    <collision>
+      <origin rpy="0 0 0" xyz="0 0 0.03585"/>
+      <geometry>
+        <cylinder radius="0.0516" length="0.0717"/>
+      </geometry>
+    </collision>
+  </link>
+  <joint name="multi_base_top_joint" type="fixed" >
+    <origin xyz="0 0 0.0377" rpy="0 0 0" />
+    <parent link="multi_base_scan" />
+    <child link="multi_top_scan"/>
+  </joint>
+  <link name="multi_top_scan">
+    <inertial>
+      <mass value="0.01"/>
+      <origin xyz="0 0 0"/>
+      <inertia ixx="1e-7" ixy="0" ixz="0" iyy="1e-7" iyz="0" izz="1e-7"/>
+    </inertial>
+    <visual>
+      <origin xyz="0 0 -0.0377" />
+      <geometry>
+        <mesh filename="package://velodyne_description/meshes/VLP16_scan.dae" scale="0.5 0.5 0.5"/>
+      </geometry>
+    </visual>
   </link>
   <joint name="camera_joint" type="fixed">

Commit message: # add kinematics

File: omtb_description/turtlebot3_description/urdf/turtlebot3_waffle.gazebo.xacro (robot description, xacro)
@@ -10,6 +10,6 @@
   </gazebo>
   <gazebo reference="wheel_left_link">
-    <mu1>1</mu1>
-    <mu2>1</mu2>
+    <mu1>1000</mu1>
+    <mu2>100</mu2>
     <kp>1000000.0</kp>
     <kd>100.0</kd>
@@ -20,6 +20,6 @@
   </gazebo>
   <gazebo reference="wheel_right_link">
-    <mu1>1</mu1>
-    <mu2>1</mu2>
+    <mu1>1000</mu1>
+    <mu2>100</mu2>
     <kp>1000000.0</kp>
     <kd>100.0</kd>
@@ -30,6 +30,6 @@
   </gazebo>
   <gazebo reference="caster_back_right_link">
-    <mu1>1</mu1>
-    <mu2>1</mu2>
+    <mu1>1000</mu1>
+    <mu2>100</mu2>
     <kp>1000000.0</kp>
     <kd>100.0</kd>
@@ -39,6 +39,6 @@
   </gazebo>
   <gazebo reference="caster_back_left_link">
-    <mu1>1</mu1>
-    <mu2>1</mu2>
+    <mu1>1000</mu1>
+    <mu2>100</mu2>
     <kp>1000000.0</kp>
     <kd>100.0</kd>
@@ -137,5 +137,5 @@
     </sensor>
   </gazebo>
-  <gazebo reference="multi_base_scan">
+  <gazebo reference="base_scan1">
     <sensor type="ray" name="VLP16">
       <pose>0 0 0 0 0 0</pose>
@@ -152,7 +152,5 @@
           <vertical>
             <samples>16</samples>
-<!--            <samples>9</samples>-->
             <resolution>1</resolution>
-<!--            <min_angle>-0.017453</min_angle>-->
             <min_angle>-0.523599</min_angle>
             <max_angle>0.523599</max_angle>
@@ -172,5 +170,5 @@
       <plugin name="gazebo_ros_laser_controller" filename="libgazebo_ros_velodyne_laser.so">
         <topicName>points2</topicName>
-        <frameName>multi_base_scan</frameName>
+        <frameName>base_scan1</frameName>
         <min_range>0.3</min_range>
         <max_range>3.5</max_range>

File: omtb_description/turtlebot3_description/urdf/turtlebot3_waffle_for_open_manipulator.urdf.xacro (robot description, xacro)
@@ -32,7 +32,7 @@
       <origin xyz="0 0 0" rpy="0 0 0"/>
       <mass value="1.3729096e+01"/>
-      <inertia ixx="8.7002718e-03" ixy="-4.7576583e-05" ixz="1.1160499e-04"
-               iyy="8.6195418e-03" iyz="-3.5422299e-06"
-               izz="1.4612727e-02" />
+      <inertia ixx="1" ixy="0" ixz="0"
+               iyy="1" iyz="0"
+               izz="1" />
     </inertial>
   </link>
@@ -180,5 +180,12 @@
     </inertial>
   </link>
-  <joint name="multi_base_mount_joint" type="fixed">
+  <joint name="scan_joint1" type="fixed">
+    <parent link="base_link"/>
+    <child link="base_scan1"/>
+    <origin xyz="-0.024 0 0.122" rpy="0 0 0"/>
+  </joint>
+  <link name="base_scan1">
+  </link>
+<!--  <joint name="multi_base_mount_joint" type="fixed">
     <parent link="base_link"/>
     <child link="multi_base_scan"/>
@@ -227,5 +234,5 @@
       </geometry>
     </visual>
-  </link>
+  </link>-->
   <joint name="camera_joint" type="fixed">
     <origin xyz="0.064 -0.065 0.094" rpy="0 0 0"/>
